File: HARDWARE/BOARD_V1/BOARD_V1.kicad_sch (KiCad schematic)
At the start: 43 parts, among them U1 STM32N657I0H3Q

Commit message: up
Other:
- sheet FLASH_RAM ports: added FLASH_CS, NRST, OCTOSPI_CLK, OCTOSPI_D0, OCTOSPI_D1, OCTOSPI_D2, OCTOSPI_D3, OCTOSPI_D4, OCTOSPI_D5, OCTOSPI_D6, OCTOSPI_D7, OCTOSPI_DQS, OCTOSPI_ECS, RAM_CS, XSPI_RST; removed none

Commit message: up
Parts:
- added C65, C66: 6pF, symbol Device:C_Small
- added C67, C68: 4pF, symbol Device:C_Small
- added R10, R11: 200R, symbol Device:R_Small
- added R12: 22R, symbol Device:R_Small
- added Y1: 830072546, 830072546, symbol samacsys2:830072546
- added Y2: 830050789, 830050789, symbol samacsys2:830050789
Connections:
- net FLASH_CS: now also U1.P13 (PN1)
- net GND: now also C65.2, C66.2, C67.2, C68.2, R10.2, R11.2, Y1.2 (GND_1)
- net OCTOSPI_CLK: now also U1.K12 (PN6)
- net OCTOSPI_D0: now also U1.L13 (PN2)
- net OCTOSPI_D1: now also U1.N13 (PN3)
- net OCTOSPI_D2: now also U1.J13 (PN4)
- net OCTOSPI_D3: now also U1.K14 (PN5)
- net OCTOSPI_D4: now also U1.J14 (PN8)
- net OCTOSPI_D5: now also U1.L14 (PN9)
- net OCTOSPI_D6: now also U1.M14 (PN10)
- net OCTOSPI_D7: now also U1.N14 (PN11)
- net OCTOSPI_DQS: now also U1.M13 (PN0)
- net RAM_CS: now also U1.J12 (PN12)
- net USB_DM1: now reaches U1.A5 (OTG1_HSDM)
- net LSE_IN: now reaches U1.B1 (PC14-OSC32_IN)
- net LSE_IN: now also C65.1, Y2.1
- net USB_DP1: now reaches U1.B5 (OTG1_HSDP)
- net LSE_OUT: now reaches U1.C1 (PC15-OSC32_OUT)
- net LSE_OUT: now also C66.1, Y2.2
- net at U1.D5 (OTG1_TXRTUNE): now also R11.1
- net CSI_D1N: now reaches U1.N2 (CSI_D1N)
- net CSI_CKN: now reaches U1.N3 (CSI_CKN)
- net CSI_D0N: now reaches U1.N4 (CSI_D0N)
- net at U1.N5 (CSI_REXT): now also R10.1
- net CSI_D1P: now reaches U1.P2 (CSI_D1P)
- net CSI_CKP: now reaches U1.P3 (CSI_CKP)
- net CSI_D0P: now reaches U1.P4 (CSI_D0P)
- net HSE_OUT: now reaches U1.A7 (PH1-OSC_OUT)
- net HSE_OUT: now also R12.2
- net HSE_IN: now reaches U1.B7 (PH0-OSC_IN)
- net HSE_IN: now also C68.1, Y1.1 (CRYSTAL_1)
- new net: C67.1, R12.1, Y1.3 (CRYSTAL_2)
- no-connect marks 0 -> 6
Other:
- sheet FLASH_RAM ports: added none; removed XSPI_RST
- note added: "32kHz 12.5pF"
- note added: "48Mhz 10pF"
- note added: "830072546"
- moved on the sheet: C1, C2, C3, C4

Commit message: up
Parts:
- added C71: 100nF, symbol Device:C_Small
Connections:
- net GND: now also C71.2
- net NRST: now also C71.1
Changed lines of the file:
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@@
 	)
 	(junction
+		(at 135.89 346.71)
+		(diameter 0)
+		(color 0 0 0 0)
+	)
+	(junction
 		(at 514.35 125.73)
 		(diameter 0)
@@
 	(wire
 		(pts
-			(xy 138.43 346.71) (xy 133.35 346.71)
+			(xy 138.43 346.71) (xy 135.89 346.71)
 		)
 		(stroke
@@
 	(wire
 		(pts
+			(xy 135.89 346.71) (xy 133.35 346.71)
+		)
+		(stroke
+			(width 0)
+			(type default)
+		)
+	)
+	(wire
+		(pts
 			(xy 59.69 336.55) (xy 62.23 336.55)
 		)
@@
 	(symbol
 		(lib_id "power:GND")
+		(at 135.89 351.79 0)
+		(unit 1)
+		(body_style 1)
+		(exclude_from_sim no)
+		(in_bom yes)
+		(on_board yes)
+		(in_pos_files yes)
+		(dnp no)
+		(fields_autoplaced yes)
+		(property "Reference" "#PWR055"
+			(at 135.89 358.14 0)
+			(hide yes)
+			(show_name no)
+			(do_not_autoplace no)
+			(effects
+				(font
+					(size 1.27 1.27)
+				)
+			)
+		)
+		(property "Value" "GND"
+			(at 135.89 356.87 0)
+			(show_name no)
+			(do_not_autoplace no)
+			(effects
+				(font
+					(size 1.27 1.27)
+				)
+			)
+		)
+		(property "Footprint" ""
+			(at 135.89 351.79 0)
+			(hide yes)
+			(show_name no)
+			(do_not_autoplace no)
+			(effects
+				(font
+					(size 1.27 1.27)
+				)
+			)
+		)
+		(property "Datasheet" ""
+			(at 135.89 351.79 0)
+			(hide yes)
+			(show_name no)
+			(do_not_autoplace no)
+			(effects
+				(font
+					(size 1.27 1.27)
+				)
+			)
+		)
+		(property "Description" "Power symbol creates a global label with name \"GND\" , ground"
+			(at 135.89 351.79 0)
+			(hide yes)
+			(show_name no)
+			(do_not_autoplace no)
+			(effects
+				(font
+					(size 1.27 1.27)
+				)
+			)
+		)
+		(pin "1"
+		)
+		(instances
+			(project "BOARD_V1"
+				(path "/8abaa504-928e-4f3c-993d-d51bf9fbdbc7"
+					(reference "#PWR055")
+					(unit 1)
+				)
+			)
+		)
+	)
+	(symbol
+		(lib_id "power:GND")
 		(at 505.46 77.47 90)
 		(unit 1)
@@
 					(unit 1)
 				)
+			)
+		)
+	)
+	(symbol
+		(lib_id "Device:C_Small")
+		(at 135.89 349.25 0)
+		(unit 1)
+		(body_style 1)
+		(exclude_from_sim no)
+		(in_bom yes)
+		(on_board yes)
+		(in_pos_files yes)
+		(dnp no)
+		(fields_autoplaced yes)
+		(property "Reference" "C71"
+			(at 138.43 347.9862 0)
+			(show_name no)
+			(do_not_autoplace no)
+			(effects
+				(font
+					(size 1.27 1.27)
+				)
+				(justify left)
+			)
+		)
+		(property "Value" "100nF"
+			(at 138.43 350.5262 0)
+			(show_name no)
+			(do_not_autoplace no)
+			(effects
+				(font
+					(size 1.27 1.27)
+				)
+				(justify left)
+			)
+		)
+		(property "Footprint" ""
+			(at 135.89 349.25 0)
+			(hide yes)
+			(show_name no)
+			(do_not_autoplace no)
+			(effects
+				(font
+					(size 1.27 1.27)
+				)
+			)
+		)
+		(property "Datasheet" ""
+			(at 135.89 349.25 0)
+			(hide yes)
+			(show_name no)
+			(do_not_autoplace no)
+			(effects
+				(font
+					(size 1.27 1.27)
+				)
+			)
+		)
+		(property "Description" "Unpolarized capacitor, small symbol"
+			(at 135.89 349.25 0)
+			(hide yes)
+			(show_name no)
+			(do_not_autoplace no)
+			(effects
+				(font
+					(size 1.27 1.27)
+				)
+			)
+		)
+		(pin "1"
+		)
+		(pin "2"
+		)
+		(instances
+			(project "BOARD_V1"
+				(path "/8abaa504-928e-4f3c-993d-d51bf9fbdbc7"
+					(reference "C71")
+					(unit 1)
+				)

Commit message: up
Connections:
- net SD_DAT0: now reaches U1.C6 (PC8)
- net SD_DAT3: now reaches U1.C7 (PC11)
- net SD_DAT1: now reaches U1.D6 (PC9)
- net SD_CLK: now reaches U1.D7 (PC12)
- net SD_DAT2: now reaches U1.D8 (PC10)
- net SD_CMD: now reaches U1.E6 (PH2)
- net CAM_SDA: now reaches U1.M7 (PA9)
- net CAM_SCL: now reaches U1.P8 (PA8)
Other:
- sheet Connector ports: added CAM_IO1, CAM_IO2, CAM_SCL, CAM_SDA, CSI_IN_CLKN, CSI_IN_CLKP, CSI_IN_D0N, CSI_IN_D0P, CSI_IN_D1N, CSI_IN_D1P, NRST, SD_CLK, SD_CMD, SD_DAT0, SD_DAT1, SD_DAT2, SD_DAT3, SD_DETECT, SWCLK, SWDIO, SWO, USB_DN, USB_DP, VBUS_SENSE; removed none
- note added: "I2C3"
- note removed: "rajouter jtag peu etre"

Commit message: up
Parts:
- added H1, H2, H3, H4: MountingHole_Pad_MP, MountingHole:MountingHole_2.2mm_M2_Pad_Via, symbol Mechanical:MountingHole_Pad_MP
- R1, R10, R11, R12: footprint (none) -> Resistor_SMD:R_0201_0603Metric_Pad0.64x0.40mm_HandSolder
- Y1: footprint 830072546 -> samacsys2:830072546
- Y2: footprint 830050789 -> samacsys2:830050789
Connections:
- net GND: now also H1.MP, H2.MP, H3.MP, H4.MP
Other:
- sheet Connector ports: added LCD_CLK, LCD_CS, LCD_DC, LCD_MOSI, LCD_PWM, LCD_RES; removed none

Commit message: up
Parts:
- removed C1: 100nF, symbol Device:C_Small
- removed C2: 1uF, symbol Device:C_Small
- removed C3: 2.2uF, symbol Device:C_Small
- removed C4: 10uF, symbol Device:C_Small
- removed L1: 2.2nH, symbol Device:L_Small
- removed L2: 1uH, symbol Device:L_Small
- added L2: LQW15AN2N2C80D, samacsys2:LQW15AN10NG80D, symbol samacsys2:LQW15AN2N2C80D
- added L5: DFE201612P-1R0M=P2, samacsys2:1286ASH1R0MP2, symbol samacsys2:DFE201612P-1R0M=P2
- C10, C11, C12, C13, C14, C15, C16, C17, C18, C19, C20, C21, C24, C25, C26, C27, C28, C29, C30, C31, C32, C5, C6, C65, C66, C67, C68, C7, C71, C8, C9: footprint (none) -> Capacitor_SMD:C_0201_0603Metric_Pad0.64x0.40mm_HandSolder
- C22, C23, C33, C34, C35, C36, C37, C38: footprint (none) -> Capacitor_SMD:C_0402_1005Metric_Pad0.74x0.62mm_HandSolder
- FB1: footprint (none) -> samacsys2:BEADC1608X100N
- U1: footprint VFBGA178_12X12_STM -> STM32N657IO:VFBGA178_12X12_STM
Connections:
- net +1V8: now also L2.2
- net VDD_CORE: now also L5.1
- net at C18.1, C19.1, C20.1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: now also L2.1
- net at R1.2, U1.G1 (VLXSMPS), U1.G2 (VLXSMPS)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: now also L5.2
Other:
- note added: "DFE201612P-1R0M"
- note added: "FBMJ1608HM180NTR"

Commit message: up
Connections:
- net JTDI: no longer names the net of U1.N12 (PA15)
- no-connect marks 6 -> 7
Other:
- sheet FLASH_RAM ports: added none; removed OCTOSPI_ECS
Changed lines of the file:
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@@
 	)
 	(no_connect
+		(at 71.12 78.74)
+	)
+	(no_connect
 		(at 62.23 341.63)
 	)
@@
 	(wire
 		(pts
-			(xy 233.68 55.88) (xy 236.22 55.88)
-		)
-		(stroke
-			(width 0)
-			(type default)
-		)
-	)
-	(wire
-		(pts
 			(xy 504.19 107.95) (xy 504.19 113.03)
 		)
@@
 	(wire
 		(pts
-			(xy 67.31 78.74) (xy 71.12 78.74)
-		)
-		(stroke
-			(width 0)
-			(type default)
-		)
-	)
-	(wire
-		(pts
 			(xy 59.69 334.01) (xy 62.23 334.01)
 		)
@@
 		)
 	)
-	(label "JTDI"
-		(at 67.31 78.74 180)
-		(effects
-			(font
-				(size 1.27 1.27)
-			)
-			(justify right bottom)
-		)
-	)
 	(label "USB_DP1"
 		(at 137.16 308.61 0)
@@
 		)
 	)
-	(label "OCTOSPI_ECS"
-		(at 233.68 55.88 180)
-		(effects
-			(font
-				(size 1.27 1.27)
-			)
-			(justify right bottom)
-		)
-	)
 	(label "SWCLK"
 		(at 67.31 76.2 180)
@@
 			(effects
 				(font
-					(size 1.27 1.27)
-				)
-				(justify left)
-			)
-		)
-		(pin "OCTOSPI_ECS" input
-			(at 236.22 55.88 180)
-			(effects
-				(font
