File: HARDWARE/BOARD_V1/BOARD_V1.kicad_sch (KiCad schematic)
At the start: 53 parts, among them U1 STM32N657I0H3Q, Y1 830072546, Y2 830050789

Commit message: up
Connections:
- net USB_DM1 renamed USB1_DN
- net USB_DP1 renamed USB1_DP
Changed lines of the file:
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@@
 		)
 	)
-	(label "USB_DP1"
+	(label "USB1_DP"
 		(at 137.16 308.61 0)
 		(effects
@@
 		)
 	)
-	(label "USB_DM1"
+	(label "USB1_DN"
 		(at 309.88 290.83 180)
 		(effects
@@
 		)
 	)
-	(label "USB_DP1"
+	(label "USB1_DP"
 		(at 309.88 287.02 180)
 		(effects
@@
 		)
 	)
-	(label "USB_DM1"
+	(label "USB1_DN"
 		(at 137.16 316.23 0)
 		(effects

Commit message: up
Parts:
- removed H1, H2, H3, H4: MountingHole_Pad_MP, MountingHole:MountingHole_2.2mm_M2_Pad_Via, symbol Mechanical:MountingHole_Pad_MP
- added H6, H7, H8, H9: MountingHole_Pad_MP, MountingHole:MountingHole_2.2mm_M2_Pad_Via, symbol Mechanical:MountingHole_Pad_MP
- added TP6: LCD, samacsys2:1mm_square, symbol Connector:TestPoint_Small
- C34: footprint Capacitor_SMD:C_0402_1005Metric_Pad0.74x0.62mm_HandSolder -> Capacitor_SMD:C_0201_0603Metric_Pad0.64x0.40mm_HandSolder
Connections:
- net BOOT_ERROR: now also TP6.1
- net CAM_IO1: now also U1.K3 (PF15)
- net CAM_IO2: now also U1.K2 (PF14)
- net FLASH_CS: now also U1.J12 (PN12); no longer U1.P13 (PN1)
- net GND: now also Y1.4 (GND_2), H6.MP, H7.MP, H8.MP, H9.MP
- net LCD_CLK: now also U1.F14 (PE2)
- net LCD_CS: now also U1.G14 (PB0)
- net LCD_DC: now also U1.D13 (PD8)
- net LCD_MOSI: now also U1.H13 (PB7)
- net LCD_PWM: now also U1.E14 (PD13)
- net LCD_RES: now also U1.C14 (PE10)
- net RAM_CS: now also U1.P13 (PN1); no longer U1.J12 (PN12)
- net SD_DETECT: now also U1.B14 (PE9)
- net USB_VBUS_SENSE: now also U1.C3 (PC13)
- net USART6_TX: now reaches U1.A8 (PC6)
- net USART6_RX: now reaches U1.A9 (PC7)
- no-connect marks 7 -> 68
Other:
- sheet Connector ports: added UART_RX, UART_TX; removed none

Commit message: up
Parts:
- removed TP6: LCD, samacsys2:1mm_square, symbol Connector:TestPoint_Small
- added C78, C82: 100nF, Capacitor_SMD:C_0201_0603Metric_Pad0.64x0.40mm_HandSolder, symbol Device:C_Small
- added LED1: APTF1616LSEEZGKQBKC, APTF1616SEEZGQBDC, symbol samacsys2:APTF1616LSEEZGKQBKC
- added R24, R26: 100R, Resistor_SMD:R_0201_0603Metric_Pad0.64x0.40mm_HandSolder, symbol Device:R_Small
- added R25: 500R, Resistor_SMD:R_0201_0603Metric_Pad0.64x0.40mm_HandSolder, symbol Device:R_Small
- added R28: 10k, Resistor_SMD:R_0201_0603Metric_Pad0.64x0.40mm_HandSolder, symbol Device:R_Small
- added S1: KXT341LHS, KXT341LHS, symbol samacsys:KXT341LHS
Connections:
- net +3.3V: now also C78.2, LED1.1 (COMMON_ANODE), S1.2 (NO)
- net BOOT0: now also C82.1, R28.2, S1.1 (COM)
- net GND: now also H6.1, H7.1, H8.1, H9.1, C78.1, C82.2, R28.1; no longer H6.MP, H7.MP, H8.MP, H9.MP
- net BLUE: now reaches U1.A13 (PD3)
- net BLUE: now also R26.2
- net GREEN: now reaches U1.B13 (PD4)
- net GREEN: now also R24.1
- net RED: now reaches U1.C13 (PE8)
- net RED: now also R25.1
- net LCD_MISO: now reaches U1.H14 (PB6)
- net NJTRST: no longer names the net of U1.L11 (PB4)
- net SWO: no longer names the net of U1.M11 (PB5)
- new net: LED1.2 (CATHODE_RED), R25.2
- new net: LED1.3 (CATHODE_GREEN), R24.2
- new net: LED1.4 (CATHODE_BLUE), R26.1
- no-connect marks 68 -> 66
Other:
- sheet Connector ports: added BOOTERR, LCD_MISO; removed SWO
- note added: "1uH R<60mohm isat > 3A"
- note added: "2mA"
- note added: "2n2H 2.53A RATED"
- note added: "BOOT0 SWITCH"
- note added: "MOUNTING_HOLE"
- note added: "RGB LED"
- note added: "STM32N657IO"
- moved on the sheet: C10, C11, C12, C13, C14, C15, C16, C17, C18, C19, C20, C21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

Commit message: up
Connections:
- net BOOT1: no longer names the net of U1.L8 (PA6)
- net VDDA1V8 renamed LDO_1V8
- no-connect marks 66 -> 70

Commit message: up
Parts:
- FB1: value FerriteBead_Small -> FBMJ1608HM180NTR
Changed lines of the file:
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@@
 			)
 		)
-		(property "Value" "FerriteBead_Small"
+		(property "Value" "FBMJ1608HM180NTR"
 			(at 444.4619 74.93 90)
 			(show_name no)

Commit message: up
Parts:
- FB1: Mouser Part Number (none) -> 963-FBMJ1608HM180NTR
Changed lines of the file:
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@@
+			)
+		)
+		(property "Mouser Part Number" "963-FBMJ1608HM180NTR"
+			(at 444.5 78.74 90)
+			(hide yes)
+			(show_name no)
+			(do_not_autoplace no)
+			(effects
+				(font
+					(size 1.27 1.27)
+				)
 			)
 		)

Commit message: up
Other:
- note added: "NCS1"
- note added: "NCS2"
Changed lines of the file:
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@@
+		)
+	)
+	(text "NCS1"
+		(exclude_from_sim no)
+		(at 163.322 60.452 0)
+		(effects
+			(font
+				(size 1.27 1.27)
+			)
 		)
 	)
@@
 		(effects
 			(font
+				(size 1.27 1.27)
+			)
+		)
+	)
+	(text "NCS2"
+		(exclude_from_sim no)
+		(at 166.37 88.138 0)
+		(effects
+			(font

Commit message: up
Parts:
- removed C82: 100nF, Capacitor_SMD:C_0201_0603Metric_Pad0.64x0.40mm_HandSolder, symbol Device:C_Small
- removed S1: KXT341LHS, KXT341LHS, symbol samacsys:KXT341LHS
- added R30: 10k, Resistor_SMD:R_0201_0603Metric_Pad0.64x0.40mm_HandSolder, symbol Device:R_Small
- added SW1: SW_DIP_x02, Button_Switch_SMD:SW_DIP_SPSTx02_Slide_KingTek_DSHP02TJ_W5.25mm_P1.27mm_JPin, symbol Switch:SW_DIP_x02
Connections:
- net BOOT0: now also SW1.2
- net GND: now also R30.1
- net VDDIO3V3: now also SW1.3, SW1.4
- net BOOT1: now reaches U1.L8 (PA6)
- net BOOT1: now also R30.2, SW1.1
- no-connect marks 70 -> 69
Other:
- moved on the sheet: R28
