File: HARDWARE/BOARD_V1/Connector.kicad_sch (KiCad schematic)
At the start: 0 parts

Commit message: up
Parts:
- added J1: SFW15R-2STE1LF, SFW15R2STE1LF, symbol samacsys2:SFW15R-2STE1LF
Changed lines of the file:
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@@
 (kicad_sch
-	(version 20250114)
+	(version 20260306)
 	(generator "eeschema")
-	(generator_version "9.0")
+	(generator_version "10.0")
 	(paper "A4")
+	(symbol
+		(lib_id "samacsys2:SFW15R-2STE1LF")
+		(at 245.11 30.48 0)
+		(mirror y)
+		(unit 1)
+		(body_style 1)
+		(exclude_from_sim no)
+		(in_bom yes)
+		(on_board yes)
+		(in_pos_files yes)
+		(dnp no)
+		(fields_autoplaced yes)
+		(property "Reference" "J1"
+			(at 232.41 22.86 0)
+			(show_name no)
+			(do_not_autoplace no)
+			(effects
+				(font
+					(size 1.27 1.27)
+				)
+			)
+		)
+		(property "Value" "SFW15R-2STE1LF"
+			(at 232.41 25.4 0)
+			(show_name no)
+			(do_not_autoplace no)
+			(effects
+				(font
+					(size 1.27 1.27)
+				)
+			)
+		)
+		(property "Footprint" "SFW15R2STE1LF"
+			(at 223.52 125.4 0)
+			(hide yes)
+			(show_name no)
+			(do_not_autoplace no)
+			(effects
+				(font
+					(size 1.27 1.27)
+				)
+				(justify left top)
+			)
+		)
+		(property "Datasheet" "https://cdn.amphenol-cs.com/media/wysiwyg/files/drawing/10172241.pdf"
+			(at 223.52 225.4 0)
+			(hide yes)
+			(show_name no)
+			(do_not_autoplace no)
+			(effects
+				(font
+					(size 1.27 1.27)
+				)
+				(justify left top)
+			)
+		)
+		(property "Description" "FFC & FPC Connectors 15P SIDE SMT ZIF UPPER CONTACT"
+			(at 245.11 30.48 0)
+			(hide yes)
+			(show_name no)
+			(do_not_autoplace no)
+			(effects
+				(font
+					(size 1.27 1.27)
+				)
+			)
+		)
+		(property "Height" "2.9"
+			(at 223.52 425.4 0)
+			(hide yes)
+			(show_name no)
+			(do_not_autoplace no)
+			(effects
+				(font
+					(size 1.27 1.27)
+				)
+				(justify left top)
+			)
+		)
+		(property "Manufacturer_Name" "Amphenol"
+			(at 223.52 525.4 0)
+			(hide yes)
+			(show_name no)
+			(do_not_autoplace no)
+			(effects
+				(font
+					(size 1.27 1.27)
+				)
+				(justify left top)
+			)
+		)
+		(property "Manufacturer_Part_Number" "SFW15R-2STE1LF"
+			(at 223.52 625.4 0)
+			(hide yes)
+			(show_name no)
+			(do_not_autoplace no)
+			(effects
+				(font
+					(size 1.27 1.27)
+				)
+				(justify left top)
+			)
+		)
+		(property "Mouser Part Number" "649-SFW15R-2STE1LF"
+			(at 223.52 725.4 0)
+			(hide yes)
+			(show_name no)
+			(do_not_autoplace no)
+			(effects
+				(font
+					(size 1.27 1.27)
+				)
+				(justify left top)
+			)
+		)
+		(property "Mouser Price/Stock" "https://www.mouser.co.uk/ProductDetail/Amphenol-FCI/SFW15R-2STE1LF?qs=XRaITl65jnu3B148xsdn9A%3D%3D"
+			(at 223.52 825.4 0)
+			(hide yes)
+			(show_name no)
+			(do_not_autoplace no)
+			(effects
+				(font
+					(size 1.27 1.27)
+				)
+				(justify left top)
+			)
+		)
+		(property "Arrow Part Number" "SFW15R-2STE1LF"
+			(at 223.52 925.4 0)
+			(hide yes)
+			(show_name no)
+			(do_not_autoplace no)
+			(effects
+				(font
+					(size 1.27 1.27)
+				)
+				(justify left top)
+			)
+		)
+		(property "Arrow Price/Stock" "https://www.arrow.com/en/products/sfw15r-2ste1lf/amphenol-fci?utm_currency=USD&region=nac"
+			(at 223.52 1025.4 0)
+			(hide yes)
+			(show_name no)
+			(do_not_autoplace no)
+			(effects
+				(font
+					(size 1.27 1.27)
+				)
+				(justify left top)
+			)
+		)
+		(pin "4"
+		)
+		(pin "11"
+		)
+		(pin "14"
+		)
+		(pin "9"
+		)
+		(pin "1"
+		)
+		(pin "2"
+		)
+		(pin "3"
+		)
+		(pin "7"
+		)
+		(pin "8"
+		)
+		(pin "6"
+		)
+		(pin "5"
+		)
+		(pin "10"
+		)
+		(pin "12"
+		)
+		(pin "13"
+		)
+		(pin "15"
+		)
+		(pin "MP1"
+		)
+		(pin "MP2"
+		)
+		(instances
+			(project "BOARD_V1"
+				(path "/8abaa504-928e-4f3c-993d-d51bf9fbdbc7/ffb1b19b-0ac7-4fc4-87ec-6e39e1378c5b"
+					(reference "J1")
+					(unit 1)
+				)
+			)
+		)
+	)
 )

Commit message: up
Parts:
- added C69, C70: 2.2uF, symbol Device:C_Small
- added D2: PMEG3050EP, SOD4725X110N, symbol samacsys2:PMEG3050EP
- added FL1, FL2, FL3, FL4: ECLAMP8052P.TCT, ECLAMP8052PTCT, symbol samacsys2:ECLAMP8052P.TCT
- added FL5: EMIF06-MSD02N16, EMIF06MSD02N16, symbol samacsys2:EMIF06-MSD02N16
- added J2: USB_C_Receptacle_USB2.0_16P, Connector_USB:USB_C_Receptacle_GCT_USB4105-xx-A_16P_TopMnt_Horizontal, symbol Connector:USB_C_Receptacle_USB2.0_16P
- added J3: 47309-2651, 473092651, symbol samacsys:47309-2651
- added J4: Conn_ARM_SWD_TagConnect_TC2030-NL, Connector:Tag-Connect_TC2030-IDC-NL_2x03_P1.27mm_Vertical, symbol Connector:Conn_ARM_SWD_TagConnect_TC2030-NL
- added R14, R15: 4.7k, symbol Device:R_Small
- added R16, R19: 22R, symbol Device:R_Small
- added R17, R18: 5.1k, symbol Device:R_Small
- added R20, R21: 100k, symbol Device:R_Small
Connections:
- net GND: now reaches J1.1
- net GND: now also J1.10, J1.4, J1.7, J1.MP1, J1.MP2, C69.2, C70.2, FL1.3 (GND), FL2.3 (GND), FL3.3 (GND), FL4.3 (GND), J2.A1 (GND), J2.A12 (GND), J2.B1 (GND), J2.B12 (GND), J2.SH (SHIELD), J4.5 (GND), R17.1, R18.1, R21.1
- net CAM_IO1: now reaches J1.11
- net CAM_IO2: now reaches J1.12
- net CAM_SCL: now reaches J1.13
- net CAM_SCL: now also R14.1
- net CAM_SDA: now reaches J1.14
- net CAM_SDA: now also R15.1
- net +3.3V: now reaches J1.15
- net +3.3V: now also C69.1, R14.2, R15.2
- net CSI_OUT_D0N: now reaches J1.2
- net CSI_OUT_D0N: now also FL1.1 (I/O+_IN)
- net CSI_OUT_D0P: now reaches J1.3
- net CSI_OUT_D0P: now also FL1.2 (I/O-_IN)
- net CSI_OUT_D1N: now reaches J1.5
- net CSI_OUT_D1N: now also FL2.1 (I/O+_IN)
- net CSI_OUT_D1P: now reaches J1.6
- net CSI_OUT_D1P: now also FL2.2 (I/O-_IN)
- net CSI_OUT_CKN: now reaches J1.8
- net CSI_OUT_CKN: now also FL3.1 (I/O+_IN)
- net CSI_OUT_CKP: now reaches J1.9
- net CSI_OUT_CKP: now also FL3.2 (I/O-_IN)
- new net: C70.1, D2.2 (A), J2.A4 (VBUS), J2.A9 (VBUS), J2.B4 (VBUS), J2.B9 (VBUS), R20.2
- new net: J2.A5 (CC1), R17.2
- new net: J2.B5 (CC2), R18.2
- new net CON_A_DN: J2.A7 (D-), J2.B7 (D-), R16.2
- new net CON_A_DP: J2.A6 (D+), J2.B6 (D+), R19.2
- new net CON_B_DN: FL4.1 (I/O+_IN), R16.1
- new net CON_B_DP: FL4.2 (I/O-_IN), R19.1
- new net CSI_IN_CLKN: FL3.5 (I/O+_OUT)
- new net CSI_IN_CLKP: FL3.4 (I/O-_OUT)
- new net CSI_IN_D0N: FL1.5 (I/O+_OUT)
- new net CSI_IN_D0P: FL1.4 (I/O-_OUT)
- new net CSI_IN_D1N: FL2.5 (I/O+_OUT)
- new net CSI_IN_D1P: FL2.4 (I/O-_OUT)
- new net NRST: J4.3 (~{RESET})
- new net SWCLK: J4.4 (SWCLK)
- new net SWDIO: J4.2 (SWDIO)
- new net SWO: J4.6 (SWO)
- new net USB_DN: FL4.5 (I/O+_OUT)
- new net USB_DP: FL4.4 (I/O-_OUT)
- new net VBUS_SENSE: R20.1, R21.2
- new net VIN: D2.1 (K), J4.1 (VCC)
- no-connect marks 0 -> 2
Other:
- moved on the sheet: J1

Commit message: up
Connections:
- net GND: now also FL5.17 (EP_(GND))
- net SD_DETECT: now reaches FL5.1 (WP/CD)
- net SD_DAT2: now reaches FL5.3 (DAT2_IN)
- net SD_DAT3: now reaches FL5.4 (DAT3_IN)
- net SD_CMD: now reaches FL5.5 (CMD_IN)
- net SD_CLK: now reaches FL5.6 (CLK_IN)
- net SD_DAT0: now reaches FL5.7 (DAT0_IN)
- net SD_DAT1: now reaches FL5.8 (DAT1_IN)
Other:
- moved on the sheet: FL5, J3

Commit message: up
Parts:
- removed FL1, FL2, FL3, FL4: ECLAMP8052P.TCT, ECLAMP8052PTCT, symbol samacsys2:ECLAMP8052P.TCT
- added C72: 4.7u, Capacitor_SMD:C_0402_1005Metric_Pad0.74x0.62mm_HandSolder, symbol Device:C_Small
- added C73, C74: 100n, Capacitor_SMD:C_0201_0603Metric, symbol Device:C_Small
- added FL6, FL7, FL8, FL9: ECMF2-40A100N6, ECMF240A100N6, symbol samacsys2:ECMF2-40A100N6
- added R40: 22R, Resistor_SMD:R_0201_0603Metric, symbol Device:R_Small
Connections:
- net +3.3V: now also FL5.15 (VCC), FL5.16 (RDATA_VCC), J3.4, C72.1, C73.1
- net CON_B_DN: now also FL9.2 (D-_TO_CONNECTOR)
- net CON_B_DP: now also FL9.1 (D+_TO_CONNECTOR)
- net CSI_IN_CLKN: now also FL8.5 (D-_TO_IC)
- net CSI_IN_CLKP: now also FL8.6 (D+_TO_IC)
- net CSI_IN_D0N: now also FL6.5 (D-_TO_IC)
- net CSI_IN_D0P: now also FL6.6 (D+_TO_IC)
- net CSI_IN_D1N: now also FL7.5 (D-_TO_IC)
- net CSI_IN_D1P: now also FL7.6 (D+_TO_IC)
- net CSI_OUT_CKN: now also FL8.2 (D-_TO_CONNECTOR)
- net CSI_OUT_CKP: now also FL8.1 (D+_TO_CONNECTOR)
- net CSI_OUT_D0N: now also FL6.2 (D-_TO_CONNECTOR)
- net CSI_OUT_D0P: now also FL6.1 (D+_TO_CONNECTOR)
- net CSI_OUT_D1N: now also FL7.2 (D-_TO_CONNECTOR)
- net CSI_OUT_D1P: now also FL7.1 (D+_TO_CONNECTOR)
- net EX_CLK: now also FL5.11 (CLK_EX), R40.1
- net EX_CMD: now also FL5.12 (CMD_EX), J3.3
- net EX_DAT0: now also FL5.10 (DAT0_EX), J3.7
- net EX_DAT1: now also FL5.9 (DAT1_EX), J3.8
- net EX_DAT2: now also FL5.14 (DAT2_EX), J3.1
- net EX_DAT3: now also FL5.13 (DAT3_EX), J3.2
- net GND: now also J3.10 (G2), J3.11 (G3), J3.6, J3.9 (G1), C72.2, C73.2, C74.2, FL6.3 (GND_1), FL6.4 (GND_2), FL7.3 (GND_1), FL7.4 (GND_2), FL8.3 (GND_1), FL8.4 (GND_2), FL9.3 (GND_1), FL9.4 (GND_2)
- net SD_DETECT: now also J3.12 (G4), C74.1
- net USB_DN: now also FL9.5 (D-_TO_IC)
- net USB_DP: now also FL9.6 (D+_TO_IC)
- net at J3.5: now also R40.2
- no-connect marks 2 -> 3
Other:
- note added: "SD_CARD"
- moved on the sheet: FL5, J3

Commit message: up
Parts:
- added C75: 1u, Capacitor_SMD:C_0402_1005Metric_Pad0.74x0.62mm_HandSolder, symbol Device:C_Small
- added C76: 10u, Capacitor_SMD:C_0402_1005Metric_Pad0.74x0.62mm_HandSolder, symbol Device:C_Small
- added J5: 687108183722, samacsys:687108183722, symbol samacsys:687108183722
- added Q1: BSS84AKQBZ, samacsys:2N7002KQBZ, symbol samacsys:2N7002KQBZ
- added R13: 33R, Resistor_SMD:R_0201_0603Metric_Pad0.64x0.40mm_HandSolder, symbol Device:R_Small
- added R22: 100R, Resistor_SMD:R_0201_0603Metric_Pad0.64x0.40mm_HandSolder, symbol Device:R_Small
- added R23: 100k, Resistor_SMD:R_0201_0603Metric_Pad0.64x0.40mm_HandSolder, symbol Device:R_Small
- added TP1, TP2, TP3, TP4, TP5, TP6, TP7, TP8, TP9: LCD, samacsys2:1mm_square, symbol Connector:TestPoint_Small
- D2: footprint SOD4725X110N -> samacsys2:SOD4725X110N
- FL5: footprint EMIF06MSD02N16 -> samacsys2:EMIF06MSD02N16
- FL6, FL7, FL8, FL9: footprint ECMF240A100N6 -> samacsys2:ECMF240A100N6
- J1: footprint SFW15R2STE1LF -> samacsys2:SFW15R2STE1LF
- J3: footprint 473092651 -> samacsys:473092651
- R14, R15, R16, R17, R18, R19, R20, R21: footprint (none) -> Resistor_SMD:R_0201_0603Metric_Pad0.64x0.40mm_HandSolder
- R40: footprint Resistor_SMD:R_0201_0603Metric -> Resistor_SMD:R_0201_0603Metric_Pad0.64x0.40mm_HandSolder
Connections:
- net +3.3V: now also C75.1, C76.1, J5.7, Q1.2 (S), R23.1, TP7.1
- net GND: now also C75.2, C76.2, J5.2, J5.MP1, J5.MP2, TP8.1
- new net: J5.1, R22.1, TP9.1
- new net: J5.6, R13.2, TP5.1
- new net: Q1.3 (D_1), Q1.4 (D_2), R22.2
- new net LCD_CLK: R13.1
- new net LCD_CS: J5.8, TP6.1
- new net LCD_DC: J5.4, TP3.1
- new net LCD_MOSI: J5.5, TP4.1
- new net LCD_PWM: Q1.1 (G), R23.2
- new net LCD_RES: J5.3, TP2.1

Commit message: up
Parts:
- C69, C70: footprint (none) -> Capacitor_SMD:C_0402_1005Metric_Pad0.74x0.62mm_HandSolder
- C72: value 4.7u -> 4.7uF
- C73, C74: value 100n -> 100nF; footprint Capacitor_SMD:C_0201_0603Metric -> Capacitor_SMD:C_0201_0603Metric_Pad0.64x0.40mm_HandSolder
- C75: value 1u -> 1uF
- C76: value 10u -> 10uF
Connections:
- net EX_CLK: now also J3.5; no longer R40.1
- net SD_CLK: now also R40.1; no longer FL5.6 (CLK_IN)
- net at R40.2: now also FL5.6 (CLK_IN); no longer J3.5
Other:
- moved on the sheet: FL5

Commit message: up
Connections:
- net CON_A_DN: now also FL9.6 (D+_TO_IC); no longer J2.A7 (D-), J2.B7 (D-)
- net CON_A_DP: now also FL9.5 (D-_TO_IC); no longer J2.A6 (D+), J2.B6 (D+)
- net CSI_IN_CLKN: now also FL8.6 (D+_TO_IC); no longer FL8.5 (D-_TO_IC)
- net CSI_IN_CLKP: now also FL8.5 (D-_TO_IC); no longer FL8.6 (D+_TO_IC)
- net CSI_IN_D0N: now also FL6.6 (D+_TO_IC); no longer FL6.5 (D-_TO_IC)
- net CSI_IN_D0P: now also FL6.5 (D-_TO_IC); no longer FL6.6 (D+_TO_IC)
- net CSI_IN_D1N: now also FL7.6 (D+_TO_IC); no longer FL7.5 (D-_TO_IC)
- net CSI_IN_D1P: now also FL7.5 (D-_TO_IC); no longer FL7.6 (D+_TO_IC)
- net CSI_OUT_CKN: now also FL8.1 (D+_TO_CONNECTOR); no longer FL8.2 (D-_TO_CONNECTOR)
- net CSI_OUT_CKP: now also FL8.2 (D-_TO_CONNECTOR); no longer FL8.1 (D+_TO_CONNECTOR)
- net CSI_OUT_D0N: now also FL6.1 (D+_TO_CONNECTOR); no longer FL6.2 (D-_TO_CONNECTOR)
- net CSI_OUT_D0P: now also FL6.2 (D-_TO_CONNECTOR); no longer FL6.1 (D+_TO_CONNECTOR)
- net CSI_OUT_D1N: now also FL7.1 (D+_TO_CONNECTOR); no longer FL7.2 (D-_TO_CONNECTOR)
- net CSI_OUT_D1P: now also FL7.2 (D-_TO_CONNECTOR); no longer FL7.1 (D+_TO_CONNECTOR)
- net USB_DN: now also R16.1; no longer FL9.5 (D-_TO_IC)
- net USB_DP: now also R19.1; no longer FL9.6 (D+_TO_IC)
- net CON_B_DN renamed CON_DP
- net CON_DP: now also J2.A6 (D+), J2.B6 (D+); no longer R16.1
- net CON_B_DP renamed CON_DN
- net CON_DN: now also J2.A7 (D-), J2.B7 (D-); no longer R19.1
Other:
- moved on the sheet: FL6, FL7, FL8, FL9

Commit message: up
Parts:
- removed TP1, TP2, TP3, TP4, TP5, TP6, TP7, TP8, TP9: LCD, samacsys2:1mm_square, symbol Connector:TestPoint_Small
- added C77: 2.2uF, Capacitor_SMD:C_0402_1005Metric_Pad0.74x0.62mm_HandSolder, symbol Device:C_Small
- added D3: PMEG3050EP, samacsys2:SOD4725X110N, symbol samacsys2:PMEG3050EP
- added FL10: ECMF2-40A100N6, samacsys2:ECMF240A100N6, symbol samacsys2:ECMF2-40A100N6
- added J6: SM04B-GHS-TB_LF__SN_, SM04B-GHS-TB, symbol samacsys:SM04B-GHS-TB_LF__SN_
- added J7: DF52-8S-0.8H_21_, DF528S08H21, symbol samacsys2:DF52-8S-0.8H_21_
- C75: footprint Capacitor_SMD:C_0402_1005Metric_Pad0.74x0.62mm_HandSolder -> Capacitor_SMD:C_0201_0603Metric_Pad0.64x0.40mm_HandSolder
- J2: footprint Connector_USB:USB_C_Receptacle_GCT_USB4105-xx-A_16P_TopMnt_Horizontal -> Connector_USB:USB_C_Receptacle_GCT_USB4110
Connections:
- net GND: now also C77.2, FL10.3 (GND_1), FL10.4 (GND_2), J6.1, J6.5 (MP), J6.6 (MP); no longer J4.5 (GND)
- net NRST: no longer J4.3 (~{RESET})
- net SWCLK: no longer J4.4 (SWCLK)
- net SWDIO: no longer J4.2 (SWDIO)
- net SWO: no longer J4.6 (SWO)
- net VIN: now also D3.1 (K); no longer J4.1 (VCC)
- new net: FL10.1 (D+_TO_CONNECTOR), J6.2
- new net: FL10.2 (D-_TO_CONNECTOR), J6.3
- new net: C77.1, D3.2 (A), J6.4
- new net UART_RX: FL10.6 (D+_TO_IC)
- new net UART_TX: FL10.5 (D-_TO_IC)
Other:
- moved on the sheet: J4
