File: HARDWARE/BOARD_V1/Connector.kicad_sch (KiCad schematic)
At the start: 36 parts, among them J1 SFW15R-2STE1LF, J2 USB_C_Receptacle_USB2.0_16P, J3 47309-2651, J4 Conn_ARM_SWD_TagConnect_TC203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, J5 687108183722, J6 SM04B-GHS-TB_LF__SN_, J7 DF52-8S-0.8H_21_, Q1 BSS84AKQBZ

Commit message: up
Parts:
- removed J4: Conn_ARM_SWD_TagConnect_TC2030-NL, Connector:Tag-Connect_TC2030-IDC-NL_2x03_P1.27mm_Vertical, symbol Connector:Conn_ARM_SWD_TagConnect_TC2030-NL
- removed J7: DF52-8S-0.8H_21_, DF528S08H21, symbol samacsys2:DF52-8S-0.8H_21_
- added J8, J9: DF52-6S-0.8H_21_, DF526S08H21, symbol samacsys2:DF52-6S-0.8H_21_
- added R27: 100R, Resistor_SMD:R_0201_0603Metric_Pad0.64x0.40mm_HandSolder, symbol Device:R_Small
Connections:
- net +3.3V: now also J8.1
- net GND: now also J8.6, J8.7 (MP_1), J8.8 (MP_2), J9.1, J9.6, J9.7 (MP_1), J9.8 (MP_2)
- net LCD_CS: now also J8.3
- net LCD_MOSI: now also J8.5
- net LCD_PWM: now also R27.1; no longer Q1.1 (G), R23.2
- net NRST: now also J9.2
- net SWCLK: now also J9.4
- net SWDIO: now also J9.5
- net CLK_RES: now reaches J5.6, R13.2
- net CLK_RES: now also J8.4
- new net: Q1.1 (G), R23.2, R27.2
- new net BOOTERR: J9.3
- new net LCD_MISO: J8.2
Other:
- note added: "CSI CAMERA (RASPBERRY PI CAM COMPATIBLE)"
- note added: "DEBUG MICRO CONNECTOR DF52 HIROSE"
- note added: "MAIN UART OUTPUT"
- note added: "SD_CARD 50Mhz max and 3.3V only"
- note added: "SECOND CONNECTOR"
- note added: "SPI DISPLAY"
- note added: "USB 2.0 USB C"
- note removed: "SD_CARD"
- moved on the sheet: C69, C70, C72, C73, C74, C75, C76, C77, D2, D3, FL10, FL5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

Commit message: up
Changed lines of the file:
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@@
-		)
-	)
-	(label "CON_B_DP"
-		(at 34.29 62.23 270)
-		(effects
-			(font
-				(size 1.27 1.27)
-			)
-			(justify right bottom)
 		)
 	)
@@
 		(effects
 			(font
-				(size 1.27 1.27)
-			)
-			(justify left bottom)
-		)
-	)
-	(label "CON_B_DN"
-		(at 34.29 59.69 90)
-		(effects
-			(font

Commit message: up
Parts:
- D2, D3: Mouser Part Number N/A -> 771-PMEG3050EP115
- J2: Mouser Part Number (none) -> 640-USB4110-GF-A
- J6: Mouser Part Number N/A -> 306-SM04BGHSTBLFSN
Changed lines of the file:
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@@
 			)
 		)
-		(property "Mouser Part Number" "N/A"
+		(property "Mouser Part Number" "771-PMEG3050EP115"
 			(at 80.01 729.21 0)
 			(hide yes)
@@
 			)
 		)
+		(property "Mouser Part Number" "640-USB4110-GF-A"
+			(at 142.24 59.69 0)
+			(hide yes)
+			(show_name no)
+			(do_not_autoplace no)
+			(effects
+				(font
+					(size 1.27 1.27)
+				)
+			)
+		)
 		(pin "B8"
 		)
@@
 			)
 		)
-		(property "Mouser Part Number" "N/A"
+		(property "Mouser Part Number" "771-PMEG3050EP115"
 			(at 115.57 -552.68 0)
 			(hide yes)
@@
 			)
 		)
-		(property "Mouser Part Number" "N/A"
+		(property "Mouser Part Number" "306-SM04BGHSTBLFSN"
 			(at 96.52 833.35 0)
 			(hide yes)
