File: HARDWARE/BOARD_V1/FLASH_RAM.kicad_sch (KiCad schematic)
At the start: 0 parts

Commit message: up
Parts:
- added C55, C56, C57, C59, C61: 100nF, symbol Device:C_Small
- added C58, C60, C62: 10uF, symbol Device:C_Small
- added C63, C64: 1uF, symbol Device:C_Small
- added D1: NSR05F30NXT5G, NSR05F30NXT5G, symbol samacsys2:NSR05F30NXT5G
- added IC6: MX25UM25645GXDI00-T, BGA24C100P5X5_800X600X120, symbol samacsys2:MX25UM25645GXDI00-T
- added IC7: APS51208N-OBR-BD, BGA24C100P5X5_600X800X120, symbol samacsys2:APS51208N-OBR-BD
- added R7: 100k, symbol Device:R_Small
- added R8, R9: 10k, symbol Device:R_Small
Connections:
- new net FLASH_CS: IC6.C2 (CS#), R9.1
- new net GND: C55.2, C56.2, C57.2, C58.2, C59.2, C60.2, C61.2, C62.2, C63.2, C64.2, IC6.B3 (GND), IC6.C1 (VSSQ_1), IC6.E5 (VSSQ_2), IC7.C1 (VSS_1), IC7.E5 (VSS_2)
- new net NRST: D1.1 (K)
- new net OCTOSPI_CLK: IC6.B2 (SCLK), IC7.B2 (CLK)
- new net OCTOSPI_D0: IC6.D3 (SIO0), IC7.D3 (ADQ0)
- new net OCTOSPI_D1: IC6.D2 (SIO1), IC7.D2 (ADQ1)
- new net OCTOSPI_D2: IC6.C4 (SIO2), IC7.C4 (ADQ2)
- new net OCTOSPI_D3: IC6.D4 (SIO3), IC7.D4 (ADQ3)
- new net OCTOSPI_D4: IC6.D5 (SIO4), IC7.D5 (ADQ4)
- new net OCTOSPI_D5: IC6.E3 (SIO5), IC7.E3 (ADQ5)
- new net OCTOSPI_D6: IC6.E2 (SIO6), IC7.E2 (ADQ6)
- new net OCTOSPI_D7: IC6.E1 (SIO7), IC7.E1 (ADQ7)
- new net OCTOSPI_DQS: IC6.C3 (DQS), IC7.C3 (DQS/DM)
- new net OCTOSPI_ECS: IC6.A5 (ECS#)
- new net RAM_CS: IC7.A3 (CE#), R8.1
- new net VDDA1V8: C55.1, C56.1, C57.1, C58.1, C59.1, C60.1, C61.1, C62.1, C63.1, C64.1, IC6.B4 (VCC), IC6.D1 (VCCQ_1), IC6.E4 (VCCQ_2), IC7.D1 (VDD_1), IC7.E4 (VDD_2), R7.2, R8.2, R9.2
- new net XSPI_RST: D1.2 (A), IC6.A4 (RESET#), IC7.A4 (RST#), R7.1
- no-connect marks 0 -> 13
Other:
- note added: "APS51208N-OBR-BD"
- note added: "MX25UM25645GXDI00"

Commit message: up
Parts:
- D1: footprint NSR05F30NXT5G -> samacsys2:NSR05F30NXT5G
- IC6: footprint BGA24C100P5X5_800X600X120 -> samacsys2:BGA24C100P5X5_800X600X120
- IC7: footprint BGA24C100P5X5_600X800X120 -> samacsys2:BGA24C100P5X5_600X800X120
- R7, R8, R9: footprint (none) -> Resistor_SMD:R_0201_0603Metric_Pad0.64x0.40mm_HandSolder
Changed lines of the file:
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@@
 			)
 		)
-		(property "Footprint" ""
+		(property "Footprint" "Resistor_SMD:R_0201_0603Metric_Pad0.64x0.40mm_HandSolder"
 			(at 99.06 50.8 0)
 			(hide yes)
@@
 			)
 		)
-		(property "Footprint" ""
+		(property "Footprint" "Resistor_SMD:R_0201_0603Metric_Pad0.64x0.40mm_HandSolder"
 			(at 115.57 55.88 0)
 			(hide yes)
@@
 			)
 		)
-		(property "Footprint" "BGA24C100P5X5_800X600X120"
+		(property "Footprint" "samacsys2:BGA24C100P5X5_800X600X120"
 			(at 156.21 214.3 0)
 			(hide yes)
@@
 			)
 		)
-		(property "Footprint" "BGA24C100P5X5_600X800X120"
+		(property "Footprint" "samacsys2:BGA24C100P5X5_600X800X120"
 			(at 156.21 150.8 0)
 			(hide yes)
@@
 			)
 		)
-		(property "Footprint" ""
+		(property "Footprint" "Resistor_SMD:R_0201_0603Metric_Pad0.64x0.40mm_HandSolder"
 			(at 104.14 142.24 0)
 			(hide yes)
@@
 			)
 		)
-		(property "Footprint" "NSR05F30NXT5G"
+		(property "Footprint" "samacsys2:NSR05F30NXT5G"
 			(at -4.75 52.07 0)
 			(hide yes)

Commit message: up
Parts:
- C55, C56, C57, C59, C61, C63, C64: footprint (none) -> Capacitor_SMD:C_0201_0603Metric_Pad0.64x0.40mm_HandSolder
- C58, C60, C62: footprint (none) -> Capacitor_SMD:C_0402_1005Metric_Pad0.74x0.62mm_HandSolder
Changed lines of the file:
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@@
 			)
 		)
-		(property "Footprint" ""
+		(property "Footprint" "Capacitor_SMD:C_0201_0603Metric_Pad0.64x0.40mm_HandSolder"
 			(at 168.91 83.82 0)
 			(hide yes)
@@
 			)
 		)
-		(property "Footprint" ""
+		(property "Footprint" "Capacitor_SMD:C_0402_1005Metric_Pad0.74x0.62mm_HandSolder"
 			(at 190.5 83.82 0)
 			(hide yes)
@@
 			)
 		)
-		(property "Footprint" ""
+		(property "Footprint" "Capacitor_SMD:C_0201_0603Metric_Pad0.64x0.40mm_HandSolder"
 			(at 168.91 147.32 0)
 			(hide yes)
@@
 			)
 		)
-		(property "Footprint" ""
+		(property "Footprint" "Capacitor_SMD:C_0201_0603Metric_Pad0.64x0.40mm_HandSolder"
 			(at 180.34 147.32 0)
 			(hide yes)
@@
 			)
 		)
-		(property "Footprint" ""
+		(property "Footprint" "Capacitor_SMD:C_0402_1005Metric_Pad0.74x0.62mm_HandSolder"
 			(at 196.85 63.5 0)
 			(hide yes)
@@
 			)
 		)
-		(property "Footprint" ""
+		(property "Footprint" "Capacitor_SMD:C_0402_1005Metric_Pad0.74x0.62mm_HandSolder"
 			(at 200.66 147.32 0)
 			(hide yes)
@@
 			)
 		)
-		(property "Footprint" ""
+		(property "Footprint" "Capacitor_SMD:C_0201_0603Metric_Pad0.64x0.40mm_HandSolder"
 			(at 185.42 63.5 0)
 			(hide yes)
@@
 			)
 		)
-		(property "Footprint" ""
+		(property "Footprint" "Capacitor_SMD:C_0201_0603Metric_Pad0.64x0.40mm_HandSolder"
 			(at 180.34 83.82 0)
 			(hide yes)
@@
 			)
 		)
-		(property "Footprint" ""
+		(property "Footprint" "Capacitor_SMD:C_0201_0603Metric_Pad0.64x0.40mm_HandSolder"
 			(at 207.01 63.5 0)
 			(hide yes)
@@
 			)
 		)
-		(property "Footprint" ""
+		(property "Footprint" "Capacitor_SMD:C_0201_0603Metric_Pad0.64x0.40mm_HandSolder"
 			(at 190.5 147.32 0)
 			(hide yes)

Commit message: up
Parts:
- IC6: footprint samacsys2:BGA24C100P5X5_800X600X120 -> samacsys2:BGA24C100P5X5_600X800X120
Connections:
- net OCTOSPI_ECS: no longer names the net of IC6.A5 (ECS#)
- no-connect marks 13 -> 14
Changed lines of the file:
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@@
+	)
+	(no_connect
+		(at 127 127)
 	)
 	(no_connect
@@
 			)
 			(justify left)
-		)
-	)
-	(hierarchical_label "OCTOSPI_ECS"
-		(shape input)
-		(at 127 127 180)
-		(effects
-			(font
-				(size 1.27 1.27)
-			)
-			(justify right)
 		)
 	)
@@
 			)
 		)
-		(property "Footprint" "samacsys2:BGA24C100P5X5_800X600X120"
+		(property "Footprint" "samacsys2:BGA24C100P5X5_600X800X120"
 			(at 156.21 214.3 0)
 			(hide yes)

Commit message: up
Parts:
- added C79, C80, C81: 10nF, Capacitor_SMD:C_0201_0603Metric_Pad0.64x0.40mm_HandSolder, symbol Device:C_Small
Connections:
- net GND: now also C79.2, C80.2, C81.2
- net VDDA1V8: now also C79.1, C80.1, C81.1
Other:
- note added: "FLASH"
- note added: "PSRAM 64Mo"
- note added: "STITCHING CAP"
- moved on the sheet: C55, C56, C57, C58, C59, C60, C61, C62, C63, C64, D1, IC6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

Commit message: up
Connections:
- net VDDA1V8 renamed LDO_1V8
Other:
- note added: "LDO_1V8 is one of the reference plane for data line between ram and flash"
Changed lines of the file:
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@@
 	(rectangle
 		(start 219.71 63.5)
-		(end 274.32 115.57)
+		(end 280.67 115.57)
 		(stroke
 			(width 0)
@@
 		)
 	)
+	(text "LDO_1V8 is one of the reference plane \nfor data line between ram and flash"
+		(exclude_from_sim no)
+		(at 249.428 101.092 0)
+		(effects
+			(font
+				(size 1.905 1.905)
+			)
+		)
+	)
 	(junction
 		(at 63.5 59.69)
@@
 		)
 	)
-	(global_label "VDDA1V8"
+	(global_label "LDO_1V8"
 		(shape input)
 		(at 90.17 52.07 90)
@@
 		)
 	)
-	(global_label "VDDA1V8"
+	(global_label "LDO_1V8"
 		(shape input)
 		(at 165.1 80.01 90)
@@
 		)
 	)
-	(global_label "VDDA1V8"
+	(global_label "LDO_1V8"
 		(shape input)
 		(at 168.91 143.51 90)
@@
 		)
 	)
-	(global_label "VDDA1V8"
+	(global_label "LDO_1V8"
 		(shape input)
 		(at 73.66 46.99 90)
@@
 		)
 	)
-	(global_label "VDDA1V8"
+	(global_label "LDO_1V8"
 		(shape input)
 		(at 78.74 138.43 90)
@@
 		)
 	)
-	(global_label "VDDA1V8"
+	(global_label "LDO_1V8"
 		(shape input)
 		(at 181.61 59.69 90)
@@
 		)
 	)
-	(global_label "VDDA1V8"
+	(global_label "LDO_1V8"
 		(shape input)
 		(at 245.11 80.01 90)
@@
 		)
 	)
-	(global_label "VDDA1V8"
+	(global_label "LDO_1V8"
 		(shape input)
 		(at 101.6 135.89 180)
@@
 		)
 	)
-	(global_label "VDDA1V8"
+	(global_label "LDO_1V8"
 		(shape input)
 		(at 134.62 123.19 0)

Commit message: up
Parts:
- IC6: Mouser Part Number (none) -> 95-25UM25645GXDI0T
- IC7: Mouser Part Number (none) -> 878-APS51208N-OBR-BD
Changed lines of the file:
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@@
 			)
 		)
-		(property "Mouser Part Number" ""
+		(property "Mouser Part Number" "95-25UM25645GXDI0T"
 			(at 130.81 813.03 0)
 			(hide yes)
@@
 			)
 		)
-		(property "Mouser Part Number" ""
+		(property "Mouser Part Number" "878-APS51208N-OBR-BD"
 			(at 130.81 749.53 0)
 			(hide yes)
