File: HARDWARE/BOARD_V1/BOARD_V1.kicad_pcb (KiCad board)
At the start: 8 copper layers, 37 x 37 mm, 137 parts, among them IC1 AP3441LSHE-7B, IC2 LDLN025M33R, IC3 LDLN025M33R, IC4 LDLN025M33R, IC5 AP3441LSHE-7B, IC6 MX25UM25645GXDI00-T, IC7 APS51208N-OBR-BD, J1 SFW15R-2STE1LF, J2 USB_C_Receptacle_USB2.0_16P, J3 47309-2651, J4 Conn_ARM_SWD_TagConnect_TC203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, J5 687108183722, Q1 BSS84AKQBZ, U1 STM32N657I0H3Q, Y1 830072546, Y2 830050789

Commit message: up
Parts:
- FL9: moved to F.Cu
- moved Y2 12.2 mm to (111.2, 122.8), turned to 0 degrees
- moved Y1 11.4 mm to (107.0, 115.2), turned to 90 degrees
- moved FL9 6.85 mm to (105.2, 121.7), turned to -90 degrees
- moved FL5 0.40 mm to (107.2, 102.7)
Routing:
- net /OCTOSPI_D7: track 31.5 -> 56.4 mm
- net /OCTOSPI_D6: track 32.4 -> 56.5 mm
- net /OCTOSPI_D5: track 32.7 -> 56.5 mm
- net /OCTOSPI_CLK: track 35.9 -> 56.4 mm
- net /OCTOSPI_D4: track 37.9 -> 56.3 mm
- net /OCTOSPI_D2: track 42.3 -> 56.3 mm
- net /OCTOSPI_D3: track 47.2 -> 56.8 mm
- net /OCTOSPI_DQS: track 52.2 -> 56.4 mm
- net /OCTOSPI_D1: track 57.3 -> 56.5 mm
- net unconnected-(IC6-ECS#-PadA5): vias 1 -> 0
- net /SD_DAT3: vias 0 -> 1
- net /SD_DAT2: vias 0 -> 1
- net /SD_DAT1: vias 0 -> 1
- net /SD_DAT0: vias 0 -> 1
- net /SD_CMD: vias 0 -> 1
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
Commit message: up
Parts:
- FL5: moved to F.Cu
- FL6, FL7, FL8: moved to B.Cu
- moved R16 118.2 mm to (107.1, 119.6), turned to -90 degrees
- moved R19 114.9 mm to (107.8, 119.6), turned to -90 degrees
- moved FB1 77.1 mm to (138.8, 122.0)
- moved L2 76.5 mm to (156.8, 108.9)
- moved L5 74.2 mm to (159.9, 113.4)
- moved C39 72.9 mm to (167.2, 103.9)
- moved C40 72.9 mm to (167.2, 105.7)
- moved C41 72.9 mm to (167.2, 107.4)
- moved C42 72.9 mm to (167.2, 109.2)
- moved C43 72.9 mm to (167.2, 110.9)
- moved C44 72.9 mm to (170.0, 103.9)
- moved C48 72.9 mm to (170.0, 105.7)
- moved C52 72.9 mm to (170.0, 107.4)
- moved C73 72.9 mm to (140.5, 91.8)
- moved C74 72.9 mm to (140.5, 93.6)
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Connections:
- FL6 pad 1: /Connector/CSI_OUT_D0P -> /Connector/CSI_OUT_D0N
- FL6 pad 2: /Connector/CSI_OUT_D0N -> /Connector/CSI_OUT_D0P
- FL6 pad 5: /CSI_D0N -> /CSI_D0P
- FL6 pad 6: /CSI_D0P -> /CSI_D0N
- FL7 pad 1: /Connector/CSI_OUT_D1P -> /Connector/CSI_OUT_D1N
- FL7 pad 2: /Connector/CSI_OUT_D1N -> /Connector/CSI_OUT_D1P
- FL7 pad 5: /CSI_D1N -> /CSI_D1P
- FL7 pad 6: /CSI_D1P -> /CSI_D1N
- FL8 pad 1: /Connector/CSI_OUT_CKP -> /Connector/CSI_OUT_CKN
- FL8 pad 2: /Connector/CSI_OUT_CKN -> /Connector/CSI_OUT_CKP
- FL8 pad 5: /CSI_CKN -> /CSI_CKP
- FL8 pad 6: /CSI_CKP -> /CSI_CKN
- FL9 pad 1: /Connector/CON_B_DP -> /Connector/CON_DN
- FL9 pad 2: /Connector/CON_B_DN -> /Connector/CON_DP
- FL9 pad 5: /USB_DM1 -> /Connector/CON_A_DP
- FL9 pad 6: /USB_DP1 -> /Connector/CON_A_DN
- J2 pad A6: /Connector/CON_A_DP -> /Connector/CON_DP
- J2 pad A7: /Connector/CON_A_DN -> /Connector/CON_DN
- J2 pad B6: /Connector/CON_A_DP -> /Connector/CON_DP
- J2 pad B7: /Connector/CON_A_DN -> /Connector/CON_DN
- R16 pad 1: /Connector/CON_B_DN -> /USB1_DN
- R19 pad 1: /Connector/CON_B_DP -> /USB1_DP
- U1 pad A5: /USB_DM1 -> /USB1_DN
- U1 pad B5: /USB_DP1 -> /USB1_DP
Routing:
- net /Connector/EX_DAT2: track 0.00 -> 5.29 mm
- net /USB1_DN: track 0.00 -> 4.98 mm
- net /Connector/EX_DAT1: track 0.00 -> 4.72 mm
- net /Connector/CON_DP: track 0.00 -> 4.62 mm
- net /USB1_DP: track 0.00 -> 4.56 mm
- net /Connector/EX_DAT3: track 0.00 -> 4.51 mm
- net /Connector/EX_DAT0: track 0.00 -> 3.91 mm
- net /Connector/CON_DN: track 0.00 -> 3.82 mm
- net /Connector/EX_CMD: track 0.00 -> 3.80 mm
- net /Connector/CON_A_DP: track 0.00 -> 3.58 mm
- net /CSI_D1N: track 0.00 -> 3.57 mm
- net /CSI_D1P: track 0.00 -> 3.53 mm
- net /OCTOSPI_D4: track 56.3 -> 53.1 mm
- net /Connector/CON_A_DN: track 0.00 -> 3.12 mm
- net /CSI_CKN: track 0.00 -> 2.88 mm
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
Commit message: up
Parts:
- removed TP1, TP2, TP3, TP4, TP5, TP7, TP8, TP9: LCD, samacsys2:1mm_square
- added C77: 2.2uF, Capacitor_SMD:C_0402_1005Metric_Pad0.74x0.62mm_HandSolder, F.Cu at (103.9, 112.5)
- added D3: PMEG3050EP, samacsys2:SOD4725X110N, F.Cu at (100.1, 113.1)
- added FL10: ECMF2-40A100N6, samacsys2:ECMF240A100N6, F.Cu at (104.8, 107.5)
- added H6: MountingHole_Pad_MP, MountingHole:MountingHole_2.2mm_M2_Pad_Via, F.Cu at (68.9, 100.5)
- added H7: MountingHole_Pad_MP, MountingHole:MountingHole_2.2mm_M2_Pad_Via, F.Cu at (68.9, 106.4)
- added H8: MountingHole_Pad_MP, MountingHole:MountingHole_2.2mm_M2_Pad_Via, F.Cu at (68.9, 112.4)
- added H9: MountingHole_Pad_MP, MountingHole:MountingHole_2.2mm_M2_Pad_Via, F.Cu at (68.9, 118.3)
- added J6: SM04B-GHS-TB_LF__SN_, samacsys:SM04B-GHS-TB, F.Cu at (101.8, 107.3)
- added J7: DF52-8S-0.8H_21_, samacsys2:DF528S08H21, F.Cu at (124.9, 94.3)
- C10, C11, C12, C13, C14, C15, C16, C17, C18, C19, C20, C21, C22, C23, C24, C25, C26, C27, C28, C29, C30, C33, C5, C55, C56, C57, C58, C59, C6, C60, C61, C62, C63, C64, C7, C71, C8, C9, FB1, R10, R11, TP6: moved to B.Cu
- C34, C75: footprint Capacitor_SMD:C_0402_1005Metric_Pad0.74x0.62mm_HandSolder -> Capacitor_SMD:C_0201_0603Metric_Pad0.64x0.40mm_HandSolder
- J2: footprint Connector_USB:USB_C_Receptacle_GCT_USB4105-xx-A_16P_TopMnt_Horizontal -> Connector_USB:USB_C_Receptacle_GCT_USB4110
- moved C58 75.9 mm to (127.9, 121.8), turned to 180 degrees
- moved C60 75.4 mm to (123.2, 113.0), turned to -90 degrees
- moved C47 74.7 mm to (107.1, 131.5), turned to 90 degrees
- moved D1 73.7 mm to (132.5, 120.7), turned to -90 degrees
- moved R9 72.7 mm to (126.5, 123.1), turned to -90 degrees
- moved IC1 72.5 mm to (109.3, 132.2), turned to -90 degrees
- moved C55 70.2 mm to (126.3, 117.7), turned to -90 degrees
- moved C56 69.7 mm to (127.8, 121.0), turned to 180 degrees
- moved R4 69.6 mm to (108.4, 130.1), turned to -90 degrees
- moved C62 69.2 mm to (127.0, 107.2)
- moved R7 68.9 mm to (132.5, 122.3), turned to -90 degrees
- moved C50 68.6 mm to (112.0, 130.1), turned to 180 degrees
- moved C64 68.1 mm to (126.8, 108.0)
- moved IC5 67.5 mm to (119.1, 130.6)
- moved C59 67.3 mm to (124.7, 112.8), turned to -90 degrees
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Connections:
- H1 pad 1: (no net) -> GND
- H2 pad 1: (no net) -> GND
- H3 pad 1: (no net) -> GND
- H4 pad 1: (no net) -> GND
- J4 pad 1: VIN -> unconnected-(J4-VCC-Pad1)
- J4 pad 2: /SWDIO -> unconnected-(J4-SWDIO-Pad2)
- J4 pad 3: /NRST -> unconnected-(J4-~{RESET}-Pad3)
- J4 pad 4: /SWCLK -> unconnected-(J4-SWCLK-Pad4)
- J4 pad 5: GND -> unconnected-(J4-GND-Pad5)
- J4 pad 6: /SWO -> unconnected-(J4-SWO-Pad6)
- TP6 pad 1: /LCD_CS -> /BOOT_ERROR
- U1 pad A8: unconnected-(U1A-PC6-PadA8) -> /USART6_TX
- U1 pad A9: unconnected-(U1A-PC7-PadA9) -> /USART6_RX
- U1 pad B14: unconnected-(U1A-PE9-PadB14) -> /SD_DETECT
- U1 pad C14: unconnected-(U1A-PE10-PadC14) -> /LCD_RES
- U1 pad C3: unconnected-(U1A-PC13-PadC3) -> /USB_VBUS_SENSE
- U1 pad D13: unconnected-(U1A-PD8-PadD13) -> /LCD_DC
- U1 pad E14: unconnected-(U1A-PD13-PadE14) -> /LCD_PWM
- U1 pad F14: unconnected-(U1A-PE2-PadF14) -> /LCD_CLK
- U1 pad G14: unconnected-(U1A-PB0-PadG14) -> /LCD_CS
- U1 pad H13: unconnected-(U1A-PB7-PadH13) -> /LCD_MOSI
- U1 pad J12: /RAM_CS -> /FLASH_CS
- U1 pad K2: unconnected-(U1A-PF14-PadK2) -> /CAM_IO2
- U1 pad K3: unconnected-(U1A-PF15-PadK3) -> /CAM_IO1
- U1 pad P13: /FLASH_CS -> /RAM_CS
- Y1 pad 4: unconnected-(Y1-GND_2-Pad4) -> GND
Routing:
- net VDDA1V8: track 1.10 -> 96.7 mm, vias 12 -> 18
- net +3.3V: track 0.66 -> 83.7 mm, vias 1 -> 15
- net VDDIO3V3: track 0.00 -> 41.1 mm, vias 6 -> 8
- net PWR_ON: track 0.00 -> 37.8 mm, vias 1 -> 4
- net /OCTOSPI_D1: track 56.1 -> 26.2 mm
- net /OCTOSPI_D2: track 56.3 -> 27.0 mm
- net VDD_CORE: track 0.00 -> 29.2 mm, vias 7 -> 11
- net /OCTOSPI_DQS: track 55.8 -> 26.5 mm
- net /OCTOSPI_D4: track 53.1 -> 24.2 mm
- net /OCTOSPI_D5: track 56.6 -> 27.8 mm
- net /OCTOSPI_D3: track 56.2 -> 28.3 mm
- net /OCTOSPI_D7: track 56.4 -> 28.7 mm
- net /SD_DETECT: track 0.00 -> 27.0 mm, vias 0 -> 2
- net /OCTOSPI_D6: track 56.5 -> 30.3 mm
- net VDD1V8AON: track 0.00 -> 25.8 mm, vias 2 -> 3
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- added copper zone on F.Cu, net +1V8
- added copper zone on F.Cu, net +3.3V
- added copper zone on B.Cu, net GND
- added copper zone on F.Cu, net GND
- added copper zone on In1.Cu, net GND
- added copper zone on In4.Cu, net GND
- added copper zone on In6.Cu, net GND
- added copper zone on B.Cu, net Net-(C18-Pad1)
- added copper zone on F.Cu, net Net-(C18-Pad1)
- added copper zone on F.Cu, net Net-(IC1-LX)
- added copper zone on F.Cu, net Net-(IC5-LX)
- added copper zone on F.Cu, net Net-(L5-Pad2)
- added copper zone on B.Cu, net Net-(U1C-VDDA18MPU)
- added copper zone on F.Cu, net VDD1V8AON
- added copper zone on B.Cu, net VDDA1V8
- added copper zone on F.Cu, net VDDA1V8
- added copper zone on B.Cu, net VDDIO3V3
- added copper zone on F.Cu, net VDDIO3V3
- added copper zone on B.Cu, net VDD_CORE
- added copper zone on F.Cu, net VDD_CORE
- added copper zone on F.Cu, net VIN

Commit message: up
Parts:
- removed H1, H2, H3, H4: MountingHole_Pad_MP, MountingHole:MountingHole_2.2mm_M2_Pad_Via
- removed J4: Conn_ARM_SWD_TagConnect_TC2030-NL, Connector:Tag-Connect_TC2030-IDC-NL_2x03_P1.27mm_Vertical
- removed J7: DF52-8S-0.8H_21_, samacsys2:DF528S08H21
- removed TP6: LCD, samacsys2:1mm_square
- added C78: 100nF, Capacitor_SMD:C_0201_0603Metric_Pad0.64x0.40mm_HandSolder, F.Cu at (105.3, 99.2)
- added C79: 10nF, Capacitor_SMD:C_0201_0603Metric_Pad0.64x0.40mm_HandSolder, F.Cu at (128.7, 107.5)
- added C80: 10nF, Capacitor_SMD:C_0201_0603Metric_Pad0.64x0.40mm_HandSolder, F.Cu at (125.2, 122.5)
- added C81: 10nF, Capacitor_SMD:C_0201_0603Metric_Pad0.64x0.40mm_HandSolder, F.Cu at (132.2, 116.3)
- added C82: 100nF, Capacitor_SMD:C_0201_0603Metric_Pad0.64x0.40mm_HandSolder, F.Cu at (106.3, 109.6)
- added J8: DF52-6S-0.8H_21_, samacsys2:DF526S08H21, F.Cu at (123.3, 98.6)
- added J9: DF52-6S-0.8H_21_, samacsys2:DF526S08H21, B.Cu at (107.4, 99.2)
- added LED1: APTF1616LSEEZGKQBKC, samacsys2:APTF1616SEEZGQBDC, F.Cu at (105.2, 101.5)
- added R24: 100R, Resistor_SMD:R_0201_0603Metric_Pad0.64x0.40mm_HandSolder, F.Cu at (105.2, 104.4)
- added R25: 500R, Resistor_SMD:R_0201_0603Metric_Pad0.64x0.40mm_HandSolder, F.Cu at (105.9, 104.4)
- added R26: 100R, Resistor_SMD:R_0201_0603Metric_Pad0.64x0.40mm_HandSolder, F.Cu at (104.5, 104.4)
- added R27: 100R, Resistor_SMD:R_0201_0603Metric_Pad0.64x0.40mm_HandSolder, F.Cu at (119.7, 103.5)
- added R28: 10k, Resistor_SMD:R_0201_0603Metric_Pad0.64x0.40mm_HandSolder, F.Cu at (106.3, 111.4)
- added S1: KXT341LHS, samacsys:KXT341LHS, F.Cu at (104.5, 110.8)
- moved H8 62.9 mm to (130.5, 100.0)
- moved H9 62.8 mm to (130.5, 130.5)
- moved H7 39.4 mm to (100.0, 130.5)
- moved H6 31.1 mm to (100.0, 100.0)
- moved C75 2.56 mm to (125.8, 101.4)
- moved C76 2.51 mm to (125.9, 102.3)
- moved C77 2.14 mm to (103.9, 114.7), turned to -90 degrees
- moved R13 1.35 mm to (122.5, 101.2), turned to 0 degrees
- moved Q1 0.91 mm to (120.8, 102.3)
- moved J5 0.88 mm to (122.1, 99.5)
- moved R22 0.88 mm to (119.7, 101.8)
- moved R7 0.50 mm to (132.0, 122.3)
- moved R23 0.40 mm to (121.0, 104.3)
- moved R8 0.23 mm to (132.0, 111.8)
- moved C73 0.19 mm to (119.0, 104.5)
Connections:
- net Net-(J5-Pad6) renamed /Connector/CLK_RES
- H6 pad 1: (no net) -> GND
- H7 pad 1: (no net) -> GND
- H8 pad 1: (no net) -> GND
- H9 pad 1: (no net) -> GND
- Q1 pad 1: /LCD_PWM -> Net-(Q1-G)
- R23 pad 2: /LCD_PWM -> Net-(Q1-G)
- U1 pad A13: unconnected-(U1A-PD3-PadA13) -> /BLUE
- U1 pad B13: unconnected-(U1A-PD4-PadB13) -> /GREEN
- U1 pad C13: unconnected-(U1A-PE8-PadC13) -> /RED
- U1 pad H14: unconnected-(U1A-PB6-PadH14) -> /LCD_MISO
- U1 pad L11: /NJTRST -> unconnected-(U1A-PB4-PadL11)
- U1 pad M11: /SWO -> unconnected-(U1A-PB5-PadM11)
Routing:
- net +3.3V: track 83.7 -> 17.4 mm, vias 15 -> 18
- net VDDA1V8: track 96.7 -> 30.5 mm, vias 18 -> 21
- net VDDIO3V3: track 41.1 -> 1.60 mm
- net /NRST: track 24.9 -> 51.8 mm, vias 2 -> 3
- net VDD_CORE: track 29.2 -> 2.68 mm
- net /SWCLK: track 0.00 -> 26.4 mm, vias 1 -> 2
- net /SWDIO: track 0.00 -> 25.1 mm, vias 1 -> 2
- net /BOOT_ERROR: track 1.37 -> 26.1 mm, vias 1 -> 2
- net /BOOT0: track 0.00 -> 21.0 mm, vias 1 -> 2
- net VIN: track 19.4 -> 0.00 mm, vias 7 -> 11
- net Net-(D2-A): track 23.2 -> 4.09 mm
- net /LCD_MISO: track 0.00 -> 15.7 mm, vias 0 -> 2
- net /BLUE: track 0.00 -> 9.19 mm
- net /RED: track 0.00 -> 9.14 mm
- net /GREEN: track 0.00 -> 8.97 mm
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- added copper zone on In3.Cu, net +3.3V
- added copper zone on In2.Cu, net GND
- added copper zone on In3.Cu, net GND
- added copper zone on In5.Cu, net GND
- added copper zone on F.Cu, net Net-(D2-A)
- added copper zone on In3.Cu, net Net-(D2-A)
- added copper zone on F.Cu, net Net-(D3-A)
- added copper zone on B.Cu, net Net-(J5-Pad1)
- added copper zone on B.Cu, net Net-(U1C-V08CAP)
- added copper zone on In3.Cu, net VDDA1V8
- added copper zone on In3.Cu, net VDDIO3V3
- added copper zone on In3.Cu, net VDD_CORE
- added copper zone on In3.Cu, net VIN
Other:
- board size 37 x 37 mm -> 37 x 37.3 mm

Commit message: up
Parts:
- added G***: LOGO, LOGO, B.Cu at (106.4, 111.3)
Connections:
- net VDDA1V8 renamed LDO_1V8
- U1 pad L8: /BOOT1 -> unconnected-(U1A-PA6-PadL8)
Other:
- board size 37 x 37.3 mm -> 37.3 x 37.3 mm
- board text added: "4.5V-5.5V M.Pommery"
- board text added: "CSI0"
- board text added: "FLASH"
- board text added: "N657"
- board text added: "PSRAM"
- board text added: "SPI"
- board text added: "ST7789"
- board text added: "SWD"
- board text added: "USB1"
- board text added: "boot0"
- board text added: "boot_err"
- board text added: "clk"
- board text added: "dio"
- board text added: "gnd"
- board text added: "nrst"
- board text added: "uSD"
- board text added: "uart6"
- board text added: "vin"

Commit message: up
Parts:
- removed C82: 100nF, Capacitor_SMD:C_0201_0603Metric_Pad0.64x0.40mm_HandSolder
- removed S1: KXT341LHS, samacsys:KXT341LHS
- added D4: LED, LED_SMD:LED_0402_1005Metric, F.Cu at (111.6, 128.3)
- added D5: LED, LED_SMD:LED_0402_1005Metric, F.Cu at (115.8, 127.5)
- added R29: 1k, Resistor_SMD:R_0201_0603Metric_Pad0.64x0.40mm_HandSolder, F.Cu at (111.5, 126.9)
- added R30: 10k, Resistor_SMD:R_0201_0603Metric_Pad0.64x0.40mm_HandSolder, B.Cu at (99.3, 122.8)
- added R31: 1k, Resistor_SMD:R_0201_0603Metric_Pad0.64x0.40mm_HandSolder, F.Cu at (115.0, 127.5)
- added SW1: SW_DIP_x02, Button_Switch_SMD:SW_DIP_SPSTx02_Slide_KingTek_DSHP02TJ_W5.25mm_P1.27mm_JPin, B.Cu at (104.5, 122.1)
- FB1: value FerriteBead_Small -> FBMJ1608HM180NTR
- R28: moved to B.Cu
- moved R28 12.2 mm to (99.3, 121.3), turned to 0 degrees
Connections:
- U1 pad L8: unconnected-(U1A-PA6-PadL8) -> /BOOT1
Routing:
- net /BOOT1: track 0.00 -> 32.9 mm, vias 0 -> 2
- net +3.3V: track 17.4 -> 7.12 mm, vias 18 -> 17
- net VDDIO3V3: track 1.60 -> 3.98 mm, vias 8 -> 9
- net +1V8: track 0.00 -> 1.82 mm
- net Net-(D4-K): track 0.00 -> 1.62 mm
- net Net-(D5-K): track 0.00 -> 0.91 mm
- net /BOOT0: track 21.0 -> 21.8 mm
- net Net-(D2-A): vias 8 -> 7
- net GND: vias 170 -> 169
Other:
- board text added: "3.3v 1.8v"
- board text added: "boot1"
