File: HARDWARE/BOARD_V1/PWR_SUPPLY.kicad_sch (KiCad schematic)
At the start: 14 parts, among them IC1 AP3441LSHE-7B, IC2 LDLN025M33R, IC3 LDLN025M33R, IC4 LDLN025M33R, IC5 AP3441LSHE-7B

Commit message: up
Parts:
- added C47, C49, C50, C51, C53, C54: 22uF, symbol Device:C_Small
- added C48, C52: 22pF, symbol Device:C_Small
- added L3, L4: 2.2uH, symbol Device:L_Small
- added R3: 91k, symbol Device:R_Small
- added R4: 20k, symbol Device:R_Small
- added R5: 200k, symbol Device:R_Small
- added R6: 100k, symbol Device:R_Small
Connections:
- net +1V8: now also C52.1, C53.1, C54.1, L4.2, R5.2
- net +3.3V: now also C48.1, C49.1, C50.1, L3.2, R3.2
- net GND: now also IC1.4 (PGND), IC1.8 (SGND), IC1.9 (EP), IC5.4 (PGND), IC5.8 (SGND), IC5.9 (EP), C47.2, C49.2, C50.2, C51.2, C53.2, C54.2, R4.1, R6.1
- net PWR_ON: now also IC1.1 (FB), IC5.1 (FB)
- net VIN: now also IC1.3 (VIN), IC5.3 (VIN), C47.1, C51.1
- net at IC1.6 (LX): now also L3.1
- net at IC5.6 (LX): now also L4.1
- new net: C48.2, R3.1, R4.2
- new net: C52.2, R5.1, R6.2
- no-connect marks 0 -> 2
Other:
- moved on the sheet: IC1

Commit message: up
Parts:
- IC1, IC5: footprint AP3441LSHE7B -> samacsys2:AP3441LSHE7B
- IC2, IC3, IC4: footprint SOT95P280X145-5N -> samacsys2:SOT95P280X145-5N
- R2, R3, R4, R5, R6: footprint (none) -> Resistor_SMD:R_0201_0603Metric_Pad0.64x0.40mm_HandSolder
Changed lines of the file:
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@@
 			)
 		)
-		(property "Footprint" "SOT95P280X145-5N"
+		(property "Footprint" "samacsys2:SOT95P280X145-5N"
 			(at 77.47 155.88 0)
 			(hide yes)
@@
 			)
 		)
-		(property "Footprint" "SOT95P280X145-5N"
+		(property "Footprint" "samacsys2:SOT95P280X145-5N"
 			(at 77.47 186.36 0)
 			(hide yes)
@@
 			)
 		)
-		(property "Footprint" "SOT95P280X145-5N"
+		(property "Footprint" "samacsys2:SOT95P280X145-5N"
 			(at 78.74 126.67 0)
 			(hide yes)
@@
 			)
 		)
-		(property "Footprint" ""
+		(property "Footprint" "Resistor_SMD:R_0201_0603Metric_Pad0.64x0.40mm_HandSolder"
 			(at 234.95 81.28 0)
 			(hide yes)
@@
 			)
 		)
-		(property "Footprint" ""
+		(property "Footprint" "Resistor_SMD:R_0201_0603Metric_Pad0.64x0.40mm_HandSolder"
 			(at 234.95 127 0)
 			(hide yes)
@@
 			)
 		)
-		(property "Footprint" ""
+		(property "Footprint" "Resistor_SMD:R_0201_0603Metric_Pad0.64x0.40mm_HandSolder"
 			(at 158.75 21.59 0)
 			(hide yes)
@@
 			)
 		)
-		(property "Footprint" "AP3441LSHE7B"
+		(property "Footprint" "samacsys2:AP3441LSHE7B"
 			(at 191.77 160.96 0)
 			(hide yes)
@@
 			)
 		)
-		(property "Footprint" "AP3441LSHE7B"
+		(property "Footprint" "samacsys2:AP3441LSHE7B"
 			(at 191.77 206.68 0)
 			(hide yes)
@@
 			)
 		)
-		(property "Footprint" ""
+		(property "Footprint" "Resistor_SMD:R_0201_0603Metric_Pad0.64x0.40mm_HandSolder"
 			(at 234.95 116.84 0)
 			(hide yes)
@@
 			)
 		)
-		(property "Footprint" ""
+		(property "Footprint" "Resistor_SMD:R_0201_0603Metric_Pad0.64x0.40mm_HandSolder"
 			(at 234.95 71.12 0)
 			(hide yes)

Commit message: up
Parts:
- removed L3, L4: 2.2uH, symbol Device:L_Small
- added L1, L4: 74479325207222, samacsys2:74479325207222, symbol samacsys2:74479325207222
- C39, C40, C41, C42, C43, C44, C48, C52: footprint (none) -> Capacitor_SMD:C_0201_0603Metric_Pad0.64x0.40mm_HandSolder
- C45, C46: footprint (none) -> Capacitor_SMD:C_0402_1005Metric_Pad0.74x0.62mm_HandSolder
- C47, C49, C50, C51, C53, C54: footprint (none) -> Capacitor_SMD:C_0603_1608Metric_Pad1.08x0.95mm_HandSolder
Connections:
- net +1V8: now also L1.2
- net +3.3V: now also L4.2
- net PWR_ON: no longer IC1.1 (FB), IC5.1 (FB)
- net at C48.2, R3.1, R4.2: now also IC1.1 (FB)
- net at C52.2, R5.1, R6.2: now also IC5.1 (FB)
- net at IC5.6 (LX): now also L1.1
- net at IC1.6 (LX): now also L4.1

Commit message: up
Other:
- note added: "2.2uH Irated > 3.5A"
- note added: "4.5V-5.5V input"
- note added: "500mA or more"
- note added: "BUCK 1V8 3A"
- note added: "BUCK 3V3 3A"
- note added: "HIGH PSRR"
- note added: "VDD1V8AON"
- note added: "VDDA1V8"
- note added: "VDDIO3V3"
- moved on the sheet: C39, C40, C41, C42, C43, C44, C45, C46, C47, C48, C49, C50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

Commit message: up
Connections:
- net VDDA1V8 renamed LDO_1V8
Other:
- note added: "LDO_1V8"
- note removed: "VDDA1V8"

Commit message: up
Parts:
- IC2, IC3, IC4: Mouser Part Number 511-LDLN025M33R -> 511-LDLN025M33R 595-TLV75518PDBVR 511-LDLN025M33R 595-TLV75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
Changed lines of the file:
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@@
 			)
 		)
-		(property "Mouser Part Number" "511-LDLN025M33R"
+		(property "Mouser Part Number" "511-LDLN025M33R 595-TLV75518PDBVR 511-LDLN025M33R 595-TLV75518PDBVR"
 			(at 77.47 785.09 0)
 			(hide yes)
@@
 			)
 		)
-		(property "Mouser Part Number" "511-LDLN025M33R"
+		(property "Mouser Part Number" "511-LDLN025M33R 595-TLV75518PDBVR 511-LDLN025M33R 595-TLV75518PDBVR"
 			(at 78.74 835.89 0)
 			(hide yes)
@@
 			)
 		)
-		(property "Mouser Part Number" "511-LDLN025M33R"
+		(property "Mouser Part Number" "511-LDLN025M33R 595-TLV75518PDBVR 511-LDLN025M33R 595-TLV75518PDBVR"
 			(at 77.47 738.1 0)
 			(hide yes)

Commit message: up
Parts:
- added D4, D5: LED, LED_SMD:LED_0402_1005Metric, symbol Device:LED
- added R29, R31: 1k, Resistor_SMD:R_0201_0603Metric_Pad0.64x0.40mm_HandSolder, symbol Device:R_Small
Connections:
- net +1V8: now also D5.2 (A)
- net +3.3V: now also D4.2 (A)
- net GND: now also R29.1, R31.1
- new net: D5.1 (K), R31.2
- new net: D4.1 (K), R29.2
